File: projects/garden_guard/PCIe-M2.kicad_sch (KiCad schematic)
At the start: 20 parts, among them M1 M.2 Solder Nut, M2 M.2 Screw, U6 AP3441SHE-7B, U7 M.2 Socket, U8 ASEK-32.768KHZ-L-R-T

Commit message: - Still working through DRC - Minor board setup tweaks
Parts:
- U6: footprint Package_DFN_QFN:DFN-8-1EP_2x2mm_P0.5mm_EP1.05x1.75mm -> Custom_DCDC:AP3441SHE-7B
Changed lines of the file:
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@@
 			)
 		)
-		(property "Footprint" "Package_DFN_QFN:DFN-8-1EP_2x2mm_P0.5mm_EP1.05x1.75mm"
+		(property "Footprint" "Custom_DCDC:AP3441SHE-7B"
 			(at 62.23 179.07 0)
 			(effects
